File: hardware/eagle/aircat.sch (EAGLE design)
At the start: 154 parts, among them CON1 A10_OLINUXINO_LIME_SHIELD_TEM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, U1 PCM3168APAP, U2 OPA1644AIPW, U3 OPA1644AIPW, U4 OPA1644AIPW, U6 LM2662M

Commit message: pads added for unused pins
Parts:
- added C76: 0.001-1µF, rcl:C-EUC0603
- added DIN2, DIN3, DIN4, DOUT2, DOUT3, MC, MDI, MDO, MODE, MS, OVF, ZERO: -5V, testpad:TPTP10SQ
- added RST: 0 Ohm, rcl:R-EU_R0603
- SV1: device con-lstb:MA03-2 -> con-lstb-without-pin-numbers:MA03-2
- SV2: value AUDIO OUTPUT -> (none); device con-lstb:MA08-2 -> con-lstb-without-pin-numbers:MA08-2
Connections:
- removed net AOP_IN_L+: U4.+IN_D
- removed net AOP_IN_L-: U4.-IN_D
- removed net DIN3(N/C): CON1_GPIO-3.18
- removed net DIN4(N/C): CON1_GPIO-3.20
- removed net N$42: U1.MDI/SDA/DEMP
- removed net N$43: U1.MDO/ADR1/MD1
- removed net VIN4+: U1.VIN4-
- removed net VIN4-: U1.VIN4+
- removed net VIN5+: U1.VIN5+
- removed net VIN5-: U1.VIN5-
- removed net VIN6+: U1.VIN6+
- removed net VIN6-: U1.VIN6-
- new net MC: MC.TP, U1.MC/SCL/FMT
- new net MDI: MDI.TP, U1.MDI/SDA/DEMP
- new net MDO: MDO.TP, U1.MDO/ADR1/MD1
- new net MODE: MODE.TP, U1.MODE
- new net MS: MS.TP, U1.MS/ADR0/MD0
- new net OVF: OVF.TP, U1.OVF
- new net VIN4-6: C76.1, U1.VIN4+, U1.VIN4-, U1.VIN5+, U1.VIN5-, U1.VIN6+, U1.VIN6-
- new net ZERO: U1.ZERO, ZERO.TP
- net +3V3: now also RST.1, RST.2
- net AOP_OUT_L: now also U4.-IN_D
- net DIN2: now also DIN2.TP
- net DIN3: now also DIN3.TP
- net DIN4: now also DIN4.TP
- net DOUT2: now also DOUT2.TP
- net DOUT3: now also DOUT3.TP
- net GND: now also C76.2, U4.+IN_D

Commit message: Mode pin connection ok (VDD+pulldown)
Parts:
- removed MC, MDI, MDO, MS: -5V, testpad:TPTP10SQ
- added R66: 220k, rcl:R-EU_R0603
- DIN2, DIN3, DIN4, DOUT2, DOUT3, ZERO: value -5V -> TPTP10SQ
- MODE: value -5V -> 0 Ohm; device testpad:TPTP10SQ -> rcl:R-EU_R0603
Connections:
- removed net MODE: MODE.TP, U1.MODE
- net +3V3: now also MODE.1, MODE.2, R66.2, U1.MODE
- net GND: now also R66.1
- net MC: now also CON1_GPIO-3.28; no longer MC.TP
- net MDI: now also CON1_GPIO-3.30; no longer MDI.TP
- net MDO: now also CON1_GPIO-3.32; no longer MDO.TP
- net MS: now also CON1_GPIO-3.26; no longer MS.TP
Other:
- moved on the sheet: DIN2, DIN3, DIN4
Changed lines of the file:
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@@
 </part>
 <part name="RST" library="rcl" deviceset="R-EU_" device="R0603" value="0 Ohm"/>
-<part name="ZERO" library="testpad" deviceset="TP" device="TP10SQ" value="-5V">
+<part name="ZERO" library="testpad" deviceset="TP" device="TP10SQ" value="">
 <attribute name="TP_SIGNAL_NAME" value=""/>
 </part>
-<part name="DOUT2" library="testpad" deviceset="TP" device="TP10SQ" value="-5V">
+<part name="DOUT2" library="testpad" deviceset="TP" device="TP10SQ" value="">
 <attribute name="TP_SIGNAL_NAME" value=""/>
 </part>
-<part name="DOUT3" library="testpad" deviceset="TP" device="TP10SQ" value="-5V">
+<part name="DOUT3" library="testpad" deviceset="TP" device="TP10SQ" value="">
 <attribute name="TP_SIGNAL_NAME" value=""/>
 </part>
-<part name="MDI" library="testpad" deviceset="TP" device="TP10SQ" value="-5V">
+<part name="DIN2" library="testpad" deviceset="TP" device="TP10SQ" value="">
 <attribute name="TP_SIGNAL_NAME" value=""/>
 </part>
-<part name="MDO" library="testpad" deviceset="TP" device="TP10SQ" value="-5V">
+<part name="DIN3" library="testpad" deviceset="TP" device="TP10SQ" value="">
 <attribute name="TP_SIGNAL_NAME" value=""/>
 </part>
-<part name="MODE" library="testpad" deviceset="TP" device="TP10SQ" value="-5V">
+<part name="DIN4" library="testpad" deviceset="TP" device="TP10SQ" value="">
 <attribute name="TP_SIGNAL_NAME" value=""/>
 </part>
-<part name="MS" library="testpad" deviceset="TP" device="TP10SQ" value="-5V">
-<attribute name="TP_SIGNAL_NAME" value=""/>
-</part>
-<part name="MC" library="testpad" deviceset="TP" device="TP10SQ" value="-5V">
-<attribute name="TP_SIGNAL_NAME" value=""/>
-</part>
-<part name="DIN2" library="testpad" deviceset="TP" device="TP10SQ" value="-5V">
-<attribute name="TP_SIGNAL_NAME" value=""/>
-</part>
-<part name="DIN3" library="testpad" deviceset="TP" device="TP10SQ" value="-5V">
-<attribute name="TP_SIGNAL_NAME" value=""/>
-</part>
-<part name="DIN4" library="testpad" deviceset="TP" device="TP10SQ" value="-5V">
-<attribute name="TP_SIGNAL_NAME" value=""/>
-</part>
+<part name="MODE" library="rcl" deviceset="R-EU_" device="R0603" value="0 Ohm"/>
+<part name="R66" library="rcl" deviceset="R-EU_" device="R0603" value="220k"/>
 </parts>
 <sheets>
@@
 <text x="152.4" y="187.96" size="7.62" layer="91">Input stage</text>
 <text x="-281.94" y="208.28" size="25.4" layer="91">AirCat</text>
+<wire x1="-236.22" y1="76.2" x2="-256.54" y2="76.2" width="0.1524" layer="98"/>
+<wire x1="-256.54" y1="76.2" x2="-256.54" y2="91.44" width="0.1524" layer="98"/>
+<wire x1="-256.54" y1="91.44" x2="-261.62" y2="91.44" width="0.1524" layer="98"/>
+<wire x1="-261.62" y1="91.44" x2="-260.604" y2="92.456" width="0.1524" layer="98"/>
+<wire x1="-261.62" y1="91.44" x2="-260.604" y2="90.424" width="0.1524" layer="98"/>
+<wire x1="-236.22" y1="73.66" x2="-259.08" y2="73.66" width="0.1524" layer="98"/>
+<wire x1="-259.08" y1="73.66" x2="-258.064" y2="74.676" width="0.1524" layer="98"/>
+<wire x1="-259.08" y1="73.66" x2="-258.064" y2="72.644" width="0.1524" layer="98"/>
 </plain>
 <instances>
@@
 <instance part="DOUT2" gate="G$1" x="-144.78" y="81.28" rot="R270"/>
 <instance part="DOUT3" gate="G$1" x="-147.32" y="78.74" rot="R270"/>
-<instance part="MDI" gate="G$1" x="-152.4" y="134.62" rot="R270"/>
-<instance part="MDO" gate="G$1" x="-154.94" y="132.08" rot="R270"/>
-<instance part="MODE" gate="G$1" x="-256.54" y="76.2" rot="R90"/>
-<instance part="MS" gate="G$1" x="-254" y="78.74" rot="R90"/>
-<instance part="MC" gate="G$1" x="-251.46" y="81.28" rot="R90"/>
-<instance part="DIN2" gate="G$1" x="-251.46" y="88.9" rot="R90"/>
-<instance part="DIN3" gate="G$1" x="-254" y="86.36" rot="R90"/>
-<instance part="DIN4" gate="G$1" x="-256.54" y="83.82" rot="R90"/>
+<instance part="DIN2" gate="G$1" x="-243.84" y="91.44" rot="R90"/>
+<instance part="DIN3" gate="G$1" x="-246.38" y="88.9" rot="R90"/>
+<instance part="DIN4" gate="G$1" x="-248.92" y="86.36" rot="R90"/>
+<instance part="MODE" gate="G$1" x="-269.24" y="86.36"/>
+<instance part="R66" gate="G$1" x="-269.24" y="96.52"/>
 </instances>
 <busses>
@@
 <label x="210.82" y="119.38" size="1.778" layer="95" rot="R180"/>
 </segment>
+<segment>
+<pinref part="R66" gate="G$1" pin="1"/>
+<wire x1="-274.32" y1="96.52" x2="-276.86" y2="96.52" width="0.1524" layer="91"/>
+<label x="-276.86" y="96.52" size="1.778" layer="95" rot="R180"/>
+</segment>
 </net>
 <net name="+5V" class="0">
@@
 <segment>
 <pinref part="U1" gate="A" pin="RST"/>
-<wire x1="-228.6" y1="73.66" x2="-261.62" y2="73.66" width="0.1524" layer="91"/>
+<wire x1="-228.6" y1="73.66" x2="-231.14" y2="73.66" width="0.1524" layer="91"/>
+<label x="-231.14" y="73.66" size="1.778" layer="95" rot="R180"/>
+</segment>
+<segment>
+<pinref part="RST" gate="G$1" pin="1"/>
+<wire x1="-271.78" y1="73.66" x2="-274.32" y2="73.66" width="0.1524" layer="91"/>
+<junction x="-271.78" y="73.66"/>
+<wire x1="-271.78" y1="77.47" x2="-271.78" y2="73.66" width="0.1524" layer="91"/>
 <pinref part="RST" gate="G$1" pin="2"/>
 <wire x1="-261.62" y1="73.66" x2="-261.62" y2="77.47" width="0.1524" layer="91"/>
 <wire x1="-261.62" y1="77.47" x2="-271.78" y2="77.47" width="0.1524" layer="91"/>
-<pinref part="RST" gate="G$1" pin="1"/>
-<wire x1="-271.78" y1="77.47" x2="-271.78" y2="73.66" width="0.1524" layer="91"/>
-<wire x1="-271.78" y1="73.66" x2="-274.32" y2="73.66" width="0.1524" layer="91"/>
-<junction x="-271.78" y="73.66"/>
-<junction x="-261.62" y="73.66"/>
 <label x="-274.32" y="73.66" size="1.778" layer="95" rot="R180"/>
-<label x="-231.14" y="73.66" size="1.778" layer="95" rot="R180"/>
+</segment>
+<segment>
+<pinref part="MODE" gate="G$1" pin="2"/>
+<wire x1="-264.16" y1="86.36" x2="-264.16" y2="91.44" width="0.1524" layer="91"/>
+<pinref part="MODE" gate="G$1" pin="1"/>
+<wire x1="-264.16" y1="91.44" x2="-274.32" y2="91.44" width="0.1524" layer="91"/>
+<wire x1="-274.32" y1="91.44" x2="-274.32" y2="86.36" width="0.1524" layer="91"/>
+<wire x1="-274.32" y1="86.36" x2="-276.86" y2="86.36" width="0.1524" layer="91"/>
+<junction x="-274.32" y="86.36"/>
+<label x="-276.86" y="86.36" size="1.778" layer="95" rot="R180"/>
+<pinref part="R66" gate="G$1" pin="2"/>
+<wire x1="-264.16" y1="91.44" x2="-264.16" y2="96.52" width="0.1524" layer="91"/>
+<junction x="-264.16" y="91.44"/>
+</segment>
+<segment>
+<pinref part="U1" gate="A" pin="MODE"/>
+<wire x1="-228.6" y1="76.2" x2="-231.14" y2="76.2" width="0.1524" layer="91"/>
+<label x="-231.14" y="76.2" size="1.778" layer="95" rot="R180"/>
 </segment>
 </net>
@@
 <segment>
 <pinref part="DIN2" gate="G$1" pin="TP"/>
-<wire x1="-248.92" y1="88.9" x2="-246.38" y2="88.9" width="0.1524" layer="91"/>
+<wire x1="-241.3" y1="91.44" x2="-238.76" y2="91.44" width="0.1524" layer="91"/>
 </segment>
 </net>
@@
 <segment>
 <pinref part="DIN3" gate="G$1" pin="TP"/>
-<wire x1="-251.46" y1="86.36" x2="-246.38" y2="86.36" width="0.1524" layer="91"/>
+<wire x1="-243.84" y1="88.9" x2="-238.76" y2="88.9" width="0.1524" layer="91"/>
 </segment>
 </net>
@@
 <segment>
 <pinref part="DIN4" gate="G$1" pin="TP"/>
-<wire x1="-254" y1="83.82" x2="-246.38" y2="83.82" width="0.1524" layer="91"/>
+<wire x1="-246.38" y1="86.36" x2="-238.76" y2="86.36" width="0.1524" layer="91"/>
 </segment>
 </net>
@@
 </segment>
 <segment>
-<pinref part="MDI" gate="G$1" pin="TP"/>
-<wire x1="-154.94" y1="134.62" x2="-160.02" y2="134.62" width="0.1524" layer="91"/>
+<pinref part="CON1" gate="_GPIO-3" pin="30"/>
+<wire x1="-182.88" y1="-15.24" x2="-180.34" y2="-15.24" width="0.1524" layer="91"/>
+<label x="-180.34" y="-15.24" size="1.778" layer="95"/>
 </segment>
 </net>
@@
 </segment>
 <segment>
-<pinref part="MDO" gate="G$1" pin="TP"/>
-<wire x1="-157.48" y1="132.08" x2="-160.02" y2="132.08" width="0.1524" layer="91"/>
-</segment>
-</net>
-<net name="MODE" class="0">
-<segment>
-<pinref part="U1" gate="A" pin="MODE"/>
-<wire x1="-228.6" y1="76.2" x2="-231.14" y2="76.2" width="0.1524" layer="91"/>
-<label x="-231.14" y="76.2" size="1.778" layer="95" rot="R180"/>
-</segment>
-<segment>
-<pinref part="MODE" gate="G$1" pin="TP"/>
-<wire x1="-254" y1="76.2" x2="-246.38" y2="76.2" width="0.1524" layer="91"/>
+<pinref part="CON1" gate="_GPIO-3" pin="32"/>
+<wire x1="-182.88" y1="-12.7" x2="-180.34" y2="-12.7" width="0.1524" layer="91"/>
+<label x="-180.34" y="-12.7" size="1.778" layer="95"/>
 </segment>
 </net>
@@
 </segment>
 <segment>
-<pinref part="MS" gate="G$1" pin="TP"/>
-<wire x1="-251.46" y1="78.74" x2="-246.38" y2="78.74" width="0.1524" layer="91"/>
+<pinref part="CON1" gate="_GPIO-3" pin="26"/>
+<wire x1="-182.88" y1="-20.32" x2="-180.34" y2="-20.32" width="0.1524" layer="91"/>
+<label x="-180.34" y="-20.32" size="1.778" layer="95"/>
 </segment>
 </net>
@@
 </segment>
 <segment>
-<pinref part="MC" gate="G$1" pin="TP"/>
-<wire x1="-248.92" y1="81.28" x2="-246.38" y2="81.28" width="0.1524" layer="91"/>
-</segment>
-</net>
+<pinref part="CON1" gate="_GPIO-3" pin="28"/>
+<wire x1="-182.88" y1="-17.78" x2="-180.34" y2="-17.78" width="0.1524" layer="91"/>
+<label x="-180.34" y="-17.78" size="1.778" layer="95"/>
+</segment>
+</net>

Commit message: added IC's part name labels
Parts:
- U1: value PCM3168APAP -> PCM3168A
Other:
- moved on the sheet: C35
Changed lines of the file:
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@@
 </classes>
 <parts>
-<part name="U1" library="pcm3168" deviceset="PCM3168APAP" device=""/>
+<part name="U1" library="pcm3168" deviceset="PCM3168APAP" device="" value="PCM3168A"/>
 <part name="U2" library="OPA1644" deviceset="OPA1644AIPW" device=""/>
 <part name="C1" library="rcl" deviceset="C-EU" device="C0603" value="10µF 16V"/>
@@
 <instance part="C33" gate="G$1" x="-210.82" y="170.18"/>
 <instance part="C34" gate="G$1" x="-203.2" y="170.18"/>
-<instance part="C35" gate="G$1" x="-223.52" y="170.18"/>
+<instance part="C35" gate="G$1" x="-238.76" y="170.18"/>
 <instance part="C36" gate="G$1" x="-231.14" y="170.18"/>
 <instance part="GND3" gate="1" x="-177.8" y="160.02"/>
@@
 <wire x1="-185.42" y1="165.1" x2="-177.8" y2="165.1" width="0.1524" layer="91"/>
 <junction x="-177.8" y="165.1"/>
-<wire x1="-170.18" y1="165.1" x2="-177.8" y2="165.1" width="0.1524" layer="91"/>
 </segment>
 <segment>
@@
 <junction x="-203.2" y="165.1"/>
 <pinref part="AGND17" gate="1" pin="GND"/>
-<wire x1="-195.58" y1="165.1" x2="-203.2" y2="165.1" width="0.1524" layer="91"/>
 </segment>
 <segment>
 <pinref part="C36" gate="G$1" pin="2"/>
 <pinref part="C35" gate="G$1" pin="2"/>
-<wire x1="-231.14" y1="165.1" x2="-223.52" y2="165.1" width="0.1524" layer="91"/>
+<wire x1="-231.14" y1="165.1" x2="-238.76" y2="165.1" width="0.1524" layer="91"/>
 <wire x1="-231.14" y1="165.1" x2="-231.14" y2="162.56" width="0.1524" layer="91"/>
 <pinref part="AGND18" gate="1" pin="GND"/>
@@
 <junction x="-203.2" y="172.72"/>
 <pinref part="P+1" gate="1" pin="+5V"/>
-<wire x1="-203.2" y1="172.72" x2="-195.58" y2="172.72" width="0.1524" layer="91"/>
 </segment>
 <segment>
 <pinref part="C36" gate="G$1" pin="1"/>
 <pinref part="C35" gate="G$1" pin="1"/>
-<wire x1="-231.14" y1="172.72" x2="-223.52" y2="172.72" width="0.1524" layer="91"/>
+<wire x1="-231.14" y1="172.72" x2="-238.76" y2="172.72" width="0.1524" layer="91"/>
 <wire x1="-231.14" y1="172.72" x2="-231.14" y2="175.26" width="0.1524" layer="91"/>
 <wire x1="-231.14" y1="175.26" x2="-231.14" y2="177.8" width="0.1524" layer="91"/>
@@
 <junction x="-177.8" y="172.72"/>
 <wire x1="-177.8" y1="172.72" x2="-185.42" y2="172.72" width="0.1524" layer="91"/>
-<wire x1="-177.8" y1="172.72" x2="-170.18" y2="172.72" width="0.1524" layer="91"/>
 </segment>
 <segment>
@@
 <wire x1="-261.62" y1="77.47" x2="-271.78" y2="77.47" width="0.1524" layer="91"/>
 <label x="-274.32" y="73.66" size="1.778" layer="95" rot="R180"/>
-</segment>
-<segment>
+<junction x="-261.62" y="73.66"/>
+</segment>
+<segment>

Commit message: change C48 capacitor
switch from C0805 to C0603 form factor and from 10µF to 100nF value.
Parts:
- C1, C11, C12, C16, C17, C2, C21, C22, C26, C27, C52, C57, C59, C6, C65, C66, C7, C70, C71: MF (none) -> AVX; MPN (none) -> 1206YD106KAT2A; OC_FARNELL (none) -> 1327727
- C10, C14, C15, C19, C20, C24, C25, C29, C30, C4, C5, C68, C69, C73, C74, C9: MF (none) -> KEMET; MPN (none) -> C0603C681J5GACTU; OC_FARNELL (none) -> 1414648
- C13, C18, C23, C28, C3, C67, C72, C8: MF (none) -> AVX; MPN (none) -> 06035C332KAT2A; OC_FARNELL (none) -> 317251
- C31, C32, C33, C34, C35, C36, C43, C44, C45, C46, C47, C51: MF (none) -> AVX; MPN (none) -> 0603ZD105KAT2A; OC_FARNELL (none) -> 1327684
- C37: MF (none) -> PANASONIC; MPN (none) -> EEEFK1V100UR; OC_FARNELL (none) -> 9695826
- C38, C39, C40, C41, C42, C75: MF (none) -> PANASONIC; MPN EEE-FK1V100UR -> EEEFK1V100UR; OC_FARNELL 9695826 -> 9695826
- C48: value 10µF -> 100nF; device rcl:C-EUC0805 -> rcl:C-EUC0603; MF (none) -> SANYO; MPN (none) -> 10SVP10M; OC_FARNELL (none) -> 9188878
- C49, C50: MF (none) -> SANYO; MPN (none) -> 10SVP10M; OC_FARNELL (none) -> 9188878
- C53, C58, C62: MF (none) -> AVX; MPN (none) -> 06035C222KAT2A; OC_FARNELL (none) -> 498592
- C54: MF (none) -> AVX; MPN (none) -> 0402YD104KAT2A; OC_FARNELL (none) -> 1327666
- C55, C56, C60, C61, C63, C64: MF (none) -> AVX; MPN (none) -> 06033C223KAT2A; OC_FARNELL (none) -> 578174
- C76, CON1, DIN2, DIN3, DIN4, DOUT2, DOUT3, MODE, R10, R11, R13, R17, R18, R20, R24, R25, R27, R3, R31, R32, R34, R38, R39, R4, R41, R44, R45, R47, R48, R50, R51, R54, R55, R57, R6, R61, R62, R64, R66, RST, SV1, SV2, TP1, TP2, TP3, TP4, ZERO: OC_FARNELL (none) -> unknown
- C77, C78: MF (none) -> AVX; MPN (none) -> 06033D104KAT2A; OC_FARNELL (none) -> 2332591
- OVF: value -5V -> TPTP10SQ; OC_FARNELL (none) -> unknown
- R1, R15, R16, R2, R22, R23, R29, R30, R36, R37, R52, R53, R59, R60, R8, R9: MF (none) -> MULTICOMP; MPN (none) -> MCRE000161; OC_FARNELL (none) -> 1711638
- R12, R14, R19, R21, R26, R28, R33, R35, R40, R42, R5, R56, R58, R63, R65, R7: MF (none) -> MULTICOMP; MPN (none) -> MCPWR05FTEW5601; OC_FARNELL (none) -> 1887301
- R43, R46, R49: MF (none) -> WERA; MPN (none) -> 167I 3K TX 9 X 80 MM; OC_FARNELL (none) -> 2213661
- U1: MF (none) -> TEXAS INSTRUMENTS; MPN (none) -> PCM3168APAP; OC_FARNELL (none) -> 1689419
- U2, U3, U4: MF (none) -> TEXAS INSTRUMENTS; MPN (none) -> OPA1644AIPW; OC_FARNELL (none) -> 1882283
- U6: MF (none) -> TEXAS INSTRUMENTS; MPN (none) -> LM2662M; OC_FARNELL (none) -> 9306803
Other:
- moved on the sheet: C48, C49, C50, C75, U6
