File: hardware/eagle/aircat.sch (EAGLE design)
At the start: 165 parts, among them CON1 A10_OLINUXINO_LIME_SHIELD_TEM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, U1 PCM3168A, U2 OPA1644AIPW, U3 OPA1644AIPW, U4 OPA1644AIPW, U6 LM2662M

Commit message: changed 10µF capa form factor
Changed 10µF 0603" package to 0805" because it's cheaper.
Minor other optimizations were made too.
Parts:
- C1, C11, C12, C16, C17, C2, C21, C22, C26, C27, C52, C57, C59, C6, C65, C66, C7, C70, C71: device rcl:C-EUC0603 -> rcl:C-EUC0805
Changed lines of the file:
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@@
 <attribute name="OC_FARNELL" value="1882283"/>
 </part>
-<part name="C1" library="rcl" deviceset="C-EU" device="C0603" value="10µF 16V">
-<attribute name="MF" value="AVX"/>
-<attribute name="MPN" value="1206YD106KAT2A"/>
-<attribute name="OC_FARNELL" value="1327727"/>
-</part>
-<part name="C2" library="rcl" deviceset="C-EU" device="C0603" value="10µF 16V">
+<part name="C1" library="rcl" deviceset="C-EU" device="C0805" value="10µF 16V">
+<attribute name="MF" value="AVX"/>
+<attribute name="MPN" value="1206YD106KAT2A"/>
+<attribute name="OC_FARNELL" value="1327727"/>
+</part>
+<part name="C2" library="rcl" deviceset="C-EU" device="C0805" value="10µF 16V">
 <attribute name="MF" value="AVX"/>
 <attribute name="MPN" value="1206YD106KAT2A"/>
@@
 <part name="AGND1" library="supply1" deviceset="GND" device=""/>
 <part name="AGND2" library="supply1" deviceset="GND" device=""/>
-<part name="C6" library="rcl" deviceset="C-EU" device="C0603" value="10µF 16V">
-<attribute name="MF" value="AVX"/>
-<attribute name="MPN" value="1206YD106KAT2A"/>
-<attribute name="OC_FARNELL" value="1327727"/>
-</part>
-<part name="C7" library="rcl" deviceset="C-EU" device="C0603" value="10µF 16V">
+<part name="C6" library="rcl" deviceset="C-EU" device="C0805" value="10µF 16V">
+<attribute name="MF" value="AVX"/>
+<attribute name="MPN" value="1206YD106KAT2A"/>
+<attribute name="OC_FARNELL" value="1327727"/>
+</part>
+<part name="C7" library="rcl" deviceset="C-EU" device="C0805" value="10µF 16V">
 <attribute name="MF" value="AVX"/>
 <attribute name="MPN" value="1206YD106KAT2A"/>
@@
 <part name="AGND4" library="supply1" deviceset="GND" device=""/>
 <part name="AGND7" library="supply1" deviceset="GND" device=""/>
-<part name="C11" library="rcl" deviceset="C-EU" device="C0603" value="10µF 16V">
-<attribute name="MF" value="AVX"/>
-<attribute name="MPN" value="1206YD106KAT2A"/>
-<attribute name="OC_FARNELL" value="1327727"/>
-</part>
-<part name="C12" library="rcl" deviceset="C-EU" device="C0603" value="10µF 16V">
+<part name="C11" library="rcl" deviceset="C-EU" device="C0805" value="10µF 16V">
+<attribute name="MF" value="AVX"/>
+<attribute name="MPN" value="1206YD106KAT2A"/>
+<attribute name="OC_FARNELL" value="1327727"/>
+</part>
+<part name="C12" library="rcl" deviceset="C-EU" device="C0805" value="10µF 16V">
 <attribute name="MF" value="AVX"/>
 <attribute name="MPN" value="1206YD106KAT2A"/>
@@
 <part name="AGND5" library="supply1" deviceset="GND" device=""/>
 <part name="AGND6" library="supply1" deviceset="GND" device=""/>
-<part name="C16" library="rcl" deviceset="C-EU" device="C0603" value="10µF 16V">
-<attribute name="MF" value="AVX"/>
-<attribute name="MPN" value="1206YD106KAT2A"/>
-<attribute name="OC_FARNELL" value="1327727"/>
-</part>
-<part name="C17" library="rcl" deviceset="C-EU" device="C0603" value="10µF 16V">
+<part name="C16" library="rcl" deviceset="C-EU" device="C0805" value="10µF 16V">
+<attribute name="MF" value="AVX"/>
+<attribute name="MPN" value="1206YD106KAT2A"/>
+<attribute name="OC_FARNELL" value="1327727"/>
+</part>
+<part name="C17" library="rcl" deviceset="C-EU" device="C0805" value="10µF 16V">
 <attribute name="MF" value="AVX"/>
 <attribute name="MPN" value="1206YD106KAT2A"/>
@@
 <part name="AGND9" library="supply1" deviceset="GND" device=""/>
 <part name="AGND10" library="supply1" deviceset="GND" device=""/>
-<part name="C21" library="rcl" deviceset="C-EU" device="C0603" value="10µF 16V">
-<attribute name="MF" value="AVX"/>
-<attribute name="MPN" value="1206YD106KAT2A"/>
-<attribute name="OC_FARNELL" value="1327727"/>
-</part>
-<part name="C22" library="rcl" deviceset="C-EU" device="C0603" value="10µF 16V">
+<part name="C21" library="rcl" deviceset="C-EU" device="C0805" value="10µF 16V">
+<attribute name="MF" value="AVX"/>
+<attribute name="MPN" value="1206YD106KAT2A"/>
+<attribute name="OC_FARNELL" value="1327727"/>
+</part>
+<part name="C22" library="rcl" deviceset="C-EU" device="C0805" value="10µF 16V">
 <attribute name="MF" value="AVX"/>
 <attribute name="MPN" value="1206YD106KAT2A"/>
@@
 <attribute name="OC_FARNELL" value="1882283"/>
 </part>
-<part name="C26" library="rcl" deviceset="C-EU" device="C0603" value="10µF 16V">
-<attribute name="MF" value="AVX"/>
-<attribute name="MPN" value="1206YD106KAT2A"/>
-<attribute name="OC_FARNELL" value="1327727"/>
-</part>
-<part name="C27" library="rcl" deviceset="C-EU" device="C0603" value="10µF 16V">
+<part name="C26" library="rcl" deviceset="C-EU" device="C0805" value="10µF 16V">
+<attribute name="MF" value="AVX"/>
+<attribute name="MPN" value="1206YD106KAT2A"/>
+<attribute name="OC_FARNELL" value="1327727"/>
+</part>
+<part name="C27" library="rcl" deviceset="C-EU" device="C0805" value="10µF 16V">
 <attribute name="MF" value="AVX"/>
 <attribute name="MPN" value="1206YD106KAT2A"/>
@@
 <part name="P+11" library="supply1" deviceset="+5V" device=""/>
 <part name="AGND20" library="supply1" deviceset="GND" device=""/>
-<part name="C52" library="rcl" deviceset="C-EU" device="C0603" value="10µF 16V">
+<part name="C52" library="rcl" deviceset="C-EU" device="C0805" value="10µF 16V">
 <attribute name="MF" value="AVX"/>
 <attribute name="MPN" value="1206YD106KAT2A"/>
@@
 <part name="AGND23" library="supply1" deviceset="GND" device=""/>
 <part name="AGND24" library="supply1" deviceset="GND" device=""/>
-<part name="C57" library="rcl" deviceset="C-EU" device="C0603" value="10µF 16V">
+<part name="C57" library="rcl" deviceset="C-EU" device="C0805" value="10µF 16V">
 <attribute name="MF" value="AVX"/>
 <attribute name="MPN" value="1206YD106KAT2A"/>
@@
 <part name="AGND26" library="supply1" deviceset="GND" device=""/>
 <part name="AGND27" library="supply1" deviceset="GND" device=""/>
-<part name="C59" library="rcl" deviceset="C-EU" device="C0603" value="10µF 16V">
+<part name="C59" library="rcl" deviceset="C-EU" device="C0805" value="10µF 16V">
 <attribute name="MF" value="AVX"/>
 <attribute name="MPN" value="1206YD106KAT2A"/>
@@
 <part name="AGND25" library="supply1" deviceset="GND" device=""/>
 <part name="AGND28" library="supply1" deviceset="GND" device=""/>
-<part name="C65" library="rcl" deviceset="C-EU" device="C0603" value="10µF 16V">
-<attribute name="MF" value="AVX"/>
-<attribute name="MPN" value="1206YD106KAT2A"/>
-<attribute name="OC_FARNELL" value="1327727"/>
-</part>
-<part name="C66" library="rcl" deviceset="C-EU" device="C0603" value="10µF 16V">
+<part name="C65" library="rcl" deviceset="C-EU" device="C0805" value="10µF 16V">
+<attribute name="MF" value="AVX"/>
+<attribute name="MPN" value="1206YD106KAT2A"/>
+<attribute name="OC_FARNELL" value="1327727"/>
+</part>
+<part name="C66" library="rcl" deviceset="C-EU" device="C0805" value="10µF 16V">
 <attribute name="MF" value="AVX"/>
 <attribute name="MPN" value="1206YD106KAT2A"/>
@@
 <part name="AGND29" library="supply1" deviceset="GND" device=""/>
 <part name="AGND30" library="supply1" deviceset="GND" device=""/>
-<part name="C70" library="rcl" deviceset="C-EU" device="C0603" value="10µF 16V">
-<attribute name="MF" value="AVX"/>
-<attribute name="MPN" value="1206YD106KAT2A"/>
-<attribute name="OC_FARNELL" value="1327727"/>
-</part>
-<part name="C71" library="rcl" deviceset="C-EU" device="C0603" value="10µF 16V">
-<attribute name="MF" value="AVX"/>
-<attribute name="MPN" value="1206YD106KAT2A"/>
+<part name="C70" library="rcl" deviceset="C-EU" device="C0805" value="10µF 16V">
+<attribute name="MF" value="AVX"/>
+<attribute name="MPN" value="1206YD106KAT2A"/>
+<attribute name="OC_FARNELL" value="1327727"/>
+</part>
+<part name="C71" library="rcl" deviceset="C-EU" device="C0805" value="10µF 16V">
+<attribute name="MF" value="AVX"/>
+<attribute name="MPN" value="1206YD106KAT2A"/>

Commit message: added power indicating led
fix #1
added green led to indicate power on the 5V rail.
Parts:
- added POWER: (no value), led:LEDSML0603
- added R67: 150, rcl:R-EU_R0603
Connections:
- new net N$38: POWER.C, R67.2
- net +5V: now also POWER.A
- net GND: now also R67.1
Changed lines of the file:
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@@
 <grid distance="0.1" unitdist="inch" unit="inch" style="lines" multiple="1" display="no" altdistance="0.01" altunitdist="inch" altunit="inch"/>
 <layers>
-<layer number="1" name="Top" color="4" fill="1" visible="yes" active="no"/>
-<layer number="2" name="Route2" color="1" fill="3" visible="yes" active="no"/>
-<layer number="3" name="Route3" color="4" fill="3" visible="yes" active="no"/>
-<layer number="4" name="Route4" color="1" fill="4" visible="yes" active="no"/>
-<layer number="5" name="Route5" color="4" fill="4" visible="yes" active="no"/>
-<layer number="6" name="Route6" color="1" fill="8" visible="yes" active="no"/>
-<layer number="7" name="Route7" color="4" fill="8" visible="yes" active="no"/>
-<layer number="8" name="Route8" color="1" fill="2" visible="yes" active="no"/>
-<layer number="9" name="Route9" color="4" fill="2" visible="yes" active="no"/>
-<layer number="10" name="Route10" color="1" fill="7" visible="yes" active="no"/>
-<layer number="11" name="Route11" color="4" fill="7" visible="yes" active="no"/>
-<layer number="12" name="Route12" color="1" fill="5" visible="yes" active="no"/>
-<layer number="13" name="Route13" color="4" fill="5" visible="yes" active="no"/>
-<layer number="14" name="Route14" color="1" fill="6" visible="yes" active="no"/>
-<layer number="15" name="Route15" color="4" fill="6" visible="yes" active="no"/>
-<layer number="16" name="Bottom" color="1" fill="1" visible="yes" active="no"/>
-<layer number="17" name="Pads" color="2" fill="1" visible="yes" active="no"/>
-<layer number="18" name="Vias" color="2" fill="1" visible="yes" active="no"/>
-<layer number="19" name="Unrouted" color="6" fill="1" visible="yes" active="no"/>
-<layer number="20" name="Dimension" color="15" fill="1" visible="yes" active="no"/>
-<layer number="21" name="tPlace" color="7" fill="1" visible="yes" active="no"/>
-<layer number="22" name="bPlace" color="7" fill="1" visible="yes" active="no"/>
-<layer number="23" name="tOrigins" color="15" fill="1" visible="yes" active="no"/>
-<layer number="24" name="bOrigins" color="15" fill="1" visible="yes" active="no"/>
-<layer number="25" name="tNames" color="7" fill="1" visible="yes" active="no"/>
-<layer number="26" name="bNames" color="7" fill="1" visible="yes" active="no"/>
-<layer number="27" name="tValues" color="7" fill="1" visible="yes" active="no"/>
-<layer number="28" name="bValues" color="7" fill="1" visible="yes" active="no"/>
+<layer number="1" name="Top" color="4" fill="1" visible="no" active="no"/>
+<layer number="2" name="Route2" color="1" fill="3" visible="no" active="no"/>
+<layer number="3" name="Route3" color="4" fill="3" visible="no" active="no"/>
+<layer number="4" name="Route4" color="1" fill="4" visible="no" active="no"/>
+<layer number="5" name="Route5" color="4" fill="4" visible="no" active="no"/>
+<layer number="6" name="Route6" color="1" fill="8" visible="no" active="no"/>
+<layer number="7" name="Route7" color="4" fill="8" visible="no" active="no"/>
+<layer number="8" name="Route8" color="1" fill="2" visible="no" active="no"/>
+<layer number="9" name="Route9" color="4" fill="2" visible="no" active="no"/>
+<layer number="10" name="Route10" color="1" fill="7" visible="no" active="no"/>
+<layer number="11" name="Route11" color="4" fill="7" visible="no" active="no"/>
+<layer number="12" name="Route12" color="1" fill="5" visible="no" active="no"/>
+<layer number="13" name="Route13" color="4" fill="5" visible="no" active="no"/>
+<layer number="14" name="Route14" color="1" fill="6" visible="no" active="no"/>
+<layer number="15" name="Route15" color="4" fill="6" visible="no" active="no"/>
+<layer number="16" name="Bottom" color="1" fill="1" visible="no" active="no"/>
+<layer number="17" name="Pads" color="2" fill="1" visible="no" active="no"/>
+<layer number="18" name="Vias" color="2" fill="1" visible="no" active="no"/>
+<layer number="19" name="Unrouted" color="6" fill="1" visible="no" active="no"/>
+<layer number="20" name="Dimension" color="15" fill="1" visible="no" active="no"/>
+<layer number="21" name="tPlace" color="7" fill="1" visible="no" active="no"/>
+<layer number="22" name="bPlace" color="7" fill="1" visible="no" active="no"/>
+<layer number="23" name="tOrigins" color="15" fill="1" visible="no" active="no"/>
+<layer number="24" name="bOrigins" color="15" fill="1" visible="no" active="no"/>
+<layer number="25" name="tNames" color="7" fill="1" visible="no" active="no"/>
+<layer number="26" name="bNames" color="7" fill="1" visible="no" active="no"/>
+<layer number="27" name="tValues" color="7" fill="1" visible="no" active="no"/>
+<layer number="28" name="bValues" color="7" fill="1" visible="no" active="no"/>
 <layer number="29" name="tStop" color="7" fill="3" visible="no" active="no"/>
 <layer number="30" name="bStop" color="7" fill="6" visible="no" active="no"/>
@@
 <layer number="35" name="tGlue" color="7" fill="4" visible="no" active="no"/>
 <layer number="36" name="bGlue" color="7" fill="5" visible="no" active="no"/>
-<layer number="37" name="tTest" color="7" fill="1" visible="yes" active="no"/>
-<layer number="38" name="bTest" color="7" fill="1" visible="yes" active="no"/>
+<layer number="37" name="tTest" color="7" fill="1" visible="no" active="no"/>
+<layer number="38" name="bTest" color="7" fill="1" visible="no" active="no"/>
 <layer number="39" name="tKeepout" color="4" fill="11" visible="no" active="no"/>
 <layer number="40" name="bKeepout" color="1" fill="11" visible="no" active="no"/>
@@
 <layer number="44" name="Drills" color="7" fill="1" visible="no" active="no"/>
 <layer number="45" name="Holes" color="7" fill="1" visible="no" active="no"/>
-<layer number="46" name="Milling" color="3" fill="1" visible="yes" active="no"/>
-<layer number="47" name="Measures" color="7" fill="1" visible="yes" active="no"/>
-<layer number="48" name="Document" color="7" fill="1" visible="yes" active="no"/>
-<layer number="49" name="Reference" color="7" fill="1" visible="yes" active="no"/>
-<layer number="50" name="dxf" color="7" fill="1" visible="yes" active="no"/>
-<layer number="51" name="tDocu" color="7" fill="1" visible="yes" active="no"/>
-<layer number="52" name="bDocu" color="7" fill="1" visible="yes" active="no"/>
-<layer number="53" name="tGND_GNDA" color="7" fill="9" visible="yes" active="no"/>
-<layer number="54" name="bGND_GNDA" color="1" fill="9" visible="yes" active="no"/>
-<layer number="56" name="wert" color="7" fill="1" visible="yes" active="no"/>
+<layer number="46" name="Milling" color="3" fill="1" visible="no" active="no"/>
+<layer number="47" name="Measures" color="7" fill="1" visible="no" active="no"/>
+<layer number="48" name="Document" color="7" fill="1" visible="no" active="no"/>
+<layer number="49" name="Reference" color="7" fill="1" visible="no" active="no"/>
+<layer number="50" name="dxf" color="7" fill="1" visible="no" active="no"/>
+<layer number="51" name="tDocu" color="7" fill="1" visible="no" active="no"/>
+<layer number="52" name="bDocu" color="7" fill="1" visible="no" active="no"/>
+<layer number="53" name="tGND_GNDA" color="7" fill="9" visible="no" active="no"/>
+<layer number="54" name="bGND_GNDA" color="1" fill="9" visible="no" active="no"/>
+<layer number="56" name="wert" color="7" fill="1" visible="no" active="no"/>
 <layer number="91" name="Nets" color="2" fill="1" visible="yes" active="yes"/>
 <layer number="92" name="Busses" color="1" fill="1" visible="yes" active="yes"/>
@@
 <attribute name="OC_FARNELL" value="unknown"/>
 </part>
+<part name="P+12" library="supply1" deviceset="+5V" device=""/>
+<part name="AGND33" library="supply1" deviceset="GND" device=""/>
+<part name="POWER" library="led" deviceset="LED" device="SML0603"/>
+<part name="R67" library="rcl" deviceset="R-EU_" device="R0603" value="150">
+<attribute name="MF" value="MULTICOMP"/>
+<attribute name="MPN" value="MCRE000161"/>
+<attribute name="OC_FARNELL" value="1711638"/>
+</part>
 </parts>
 <sheets>
@@
 <attribute name="MPN" x="-269.24" y="96.52" size="1.778" layer="96" display="off"/>
 </instance>
+<instance part="P+12" gate="1" x="-256.54" y="-88.9"/>
+<instance part="AGND33" gate="1" x="-256.54" y="-119.38" smashed="yes">
+<attribute name="VALUE" x="-259.08" y="-121.92" size="1.778" layer="96"/>
+</instance>
+<instance part="POWER" gate="G$1" x="-256.54" y="-96.52"/>
+<instance part="R67" gate="G$1" x="-256.54" y="-109.22" rot="R90">
+<attribute name="OC_FARNELL" x="-256.54" y="-111.76" size="1.778" layer="96" rot="R90" display="off"/>
+<attribute name="MF" x="-256.54" y="-111.76" size="1.778" layer="96" rot="R90" display="off"/>
+<attribute name="MPN" x="-256.54" y="-111.76" size="1.778" layer="96" rot="R90" display="off"/>
+</instance>
 </instances>
 <busses>
@@
 <label x="-276.86" y="96.52" size="1.778" layer="95" rot="R180"/>
 </segment>
+<segment>
+<pinref part="R67" gate="G$1" pin="1"/>
+<pinref part="AGND33" gate="1" pin="GND"/>
+<wire x1="-256.54" y1="-116.84" x2="-256.54" y2="-114.3" width="0.1524" layer="91"/>
+</segment>
 </net>
 <net name="+5V" class="0">
@@
 <label x="-210.82" y="-119.38" size="1.778" layer="95" rot="R180"/>
 </segment>
+<segment>
+<pinref part="P+12" gate="1" pin="+5V"/>
+<pinref part="POWER" gate="G$1" pin="A"/>
+<wire x1="-256.54" y1="-91.44" x2="-256.54" y2="-93.98" width="0.1524" layer="91"/>
+</segment>
 </net>
 <net name="+3V3" class="0">
@@
 </segment>
 </net>
+<net name="N$38" class="0">
+<segment>
+<pinref part="POWER" gate="G$1" pin="C"/>
+<pinref part="R67" gate="G$1" pin="2"/>
+<wire x1="-256.54" y1="-104.14" x2="-256.54" y2="-101.6" width="0.1524" layer="91"/>
+</segment>
+</net>
