File: hardware/eagle/aircat.sch (EAGLE design)
At the start: 167 parts, among them CON1 A10_OLINUXINO_LIME_SHIELD_TEM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, U1 PCM3168A, U2 OPA1644AIPW, U3 OPA1644AIPW, U4 OPA1644AIPW, U6 LM2662M

Commit message: added SPDIF OUT connector
fix #4
Parts:
- added CON4: SPDIF_OUT, con-lstb-without-pin-numbers:MA02-1
- CON2: value (none) -> ANALOG_OUT
- CON3: value (none) -> ANALOG_IN
- renumbered SV1 to CON3, SV2 to CON2
Connections:
- new net SPDIF_DO: CON1_GPIO-3.24, CON4.2
- net GND: now also CON4.1
Changed lines of the file:
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@@
 <attribute name="OC_FARNELL" value="unknown"/>
 </part>
-<part name="SV1" library="con-lstb-without-pin-numbers" deviceset="MA03-2" device="">
+<part name="CON3" library="con-lstb-without-pin-numbers" deviceset="MA03-2" device="" value="ANALOG_IN">
 <attribute name="MF" value=""/>
 <attribute name="MPN" value=""/>
 <attribute name="OC_FARNELL" value="unknown"/>
 </part>
-<part name="SV2" library="con-lstb-without-pin-numbers" deviceset="MA08-2" device="">
+<part name="CON2" library="con-lstb-without-pin-numbers" deviceset="MA08-2" device="" value="ANALOG_OUT">
 <attribute name="MF" value=""/>
 <attribute name="MPN" value=""/>
@@
 <attribute name="OC_FARNELL" value="1711638"/>
 </part>
+<part name="CON4" library="con-lstb-without-pin-numbers" deviceset="MA02-1" device="" value="SPDIF_OUT"/>
 </parts>
 <sheets>
@@
 <attribute name="MPN" x="-195.58" y="-114.3" size="1.778" layer="96" display="off"/>
 </instance>
-<instance part="SV1" gate="1" x="246.38" y="180.34"/>
-<instance part="SV2" gate="G$1" x="-50.8" y="170.18"/>
+<instance part="CON3" gate="1" x="246.38" y="180.34"/>
+<instance part="CON2" gate="G$1" x="-50.8" y="170.18"/>
 <instance part="C76" gate="G$1" x="269.24" y="-124.46">
 <attribute name="OC_FARNELL" x="269.24" y="-124.46" size="1.778" layer="96" display="off"/>
@@
 <attribute name="MPN" x="-256.54" y="-111.76" size="1.778" layer="96" rot="R90" display="off"/>
 </instance>
+<instance part="CON4" gate="G$1" x="-152.4" y="-5.08"/>
 </instances>
 <busses>
@@
 <wire x1="-58.42" y1="180.34" x2="-60.96" y2="180.34" width="0.1524" layer="91"/>
 <label x="-60.96" y="180.34" size="1.778" layer="95" rot="R180"/>
-<pinref part="SV2" gate="G$1" pin="16"/>
+<pinref part="CON2" gate="G$1" pin="16"/>
 </segment>
 </net>
@@
 <wire x1="-58.42" y1="177.8" x2="-60.96" y2="177.8" width="0.1524" layer="91"/>
 <label x="-60.96" y="177.8" size="1.778" layer="95" rot="R180"/>
-<pinref part="SV2" gate="G$1" pin="14"/>
+<pinref part="CON2" gate="G$1" pin="14"/>
 </segment>
 </net>
@@
 <wire x1="-58.42" y1="175.26" x2="-60.96" y2="175.26" width="0.1524" layer="91"/>
 <label x="-60.96" y="175.26" size="1.778" layer="95" rot="R180"/>
-<pinref part="SV2" gate="G$1" pin="12"/>
+<pinref part="CON2" gate="G$1" pin="12"/>
 </segment>
 <segment>
@@
 <wire x1="-58.42" y1="172.72" x2="-60.96" y2="172.72" width="0.1524" layer="91"/>
 <label x="-60.96" y="172.72" size="1.778" layer="95" rot="R180"/>
-<pinref part="SV2" gate="G$1" pin="10"/>
+<pinref part="CON2" gate="G$1" pin="10"/>
 </segment>
 <segment>
@@
 <wire x1="-58.42" y1="170.18" x2="-60.96" y2="170.18" width="0.1524" layer="91"/>
 <label x="-60.96" y="170.18" size="1.778" layer="95" rot="R180"/>
-<pinref part="SV2" gate="G$1" pin="8"/>
+<pinref part="CON2" gate="G$1" pin="8"/>
 </segment>
 <segment>
@@
 <wire x1="-58.42" y1="167.64" x2="-60.96" y2="167.64" width="0.1524" layer="91"/>
 <label x="-60.96" y="167.64" size="1.778" layer="95" rot="R180"/>
-<pinref part="SV2" gate="G$1" pin="6"/>
+<pinref part="CON2" gate="G$1" pin="6"/>
 </segment>
 <segment>
@@
 <wire x1="-58.42" y1="165.1" x2="-60.96" y2="165.1" width="0.1524" layer="91"/>
 <label x="-60.96" y="165.1" size="1.778" layer="95" rot="R180"/>
-<pinref part="SV2" gate="G$1" pin="4"/>
+<pinref part="CON2" gate="G$1" pin="4"/>
 </segment>
 <segment>
@@
 <wire x1="-58.42" y1="162.56" x2="-60.96" y2="162.56" width="0.1524" layer="91"/>
 <label x="-60.96" y="162.56" size="1.778" layer="95" rot="R180"/>
-<pinref part="SV2" gate="G$1" pin="2"/>
+<pinref part="CON2" gate="G$1" pin="2"/>
 </segment>
 <segment>
@@
 <wire x1="-43.18" y1="175.26" x2="-43.18" y2="177.8" width="0.1524" layer="91"/>
 <wire x1="-43.18" y1="177.8" x2="-43.18" y2="180.34" width="0.1524" layer="91"/>
-<pinref part="SV2" gate="G$1" pin="1"/>
+<pinref part="CON2" gate="G$1" pin="1"/>
 <junction x="-43.18" y="162.56"/>
-<pinref part="SV2" gate="G$1" pin="3"/>
+<pinref part="CON2" gate="G$1" pin="3"/>
 <junction x="-43.18" y="165.1"/>
-<pinref part="SV2" gate="G$1" pin="5"/>
+<pinref part="CON2" gate="G$1" pin="5"/>
 <junction x="-43.18" y="167.64"/>
-<pinref part="SV2" gate="G$1" pin="7"/>
+<pinref part="CON2" gate="G$1" pin="7"/>
 <junction x="-43.18" y="170.18"/>
-<pinref part="SV2" gate="G$1" pin="9"/>
+<pinref part="CON2" gate="G$1" pin="9"/>
 <junction x="-43.18" y="172.72"/>
-<pinref part="SV2" gate="G$1" pin="11"/>
+<pinref part="CON2" gate="G$1" pin="11"/>
 <junction x="-43.18" y="175.26"/>
-<pinref part="SV2" gate="G$1" pin="13"/>
+<pinref part="CON2" gate="G$1" pin="13"/>
 <junction x="-43.18" y="177.8"/>
-<pinref part="SV2" gate="G$1" pin="15"/>
+<pinref part="CON2" gate="G$1" pin="15"/>
 </segment>
 <segment>
@@
 <junction x="256.54" y="180.34"/>
 <junction x="256.54" y="177.8"/>
-<pinref part="SV1" gate="1" pin="1"/>
-<pinref part="SV1" gate="1" pin="3"/>
-<pinref part="SV1" gate="1" pin="5"/>
+<pinref part="CON3" gate="1" pin="1"/>
+<pinref part="CON3" gate="1" pin="3"/>
+<pinref part="CON3" gate="1" pin="5"/>
 </segment>
 <segment>
@@
 <wire x1="-256.54" y1="-116.84" x2="-256.54" y2="-114.3" width="0.1524" layer="91"/>
 </segment>
+<segment>
+<pinref part="CON4" gate="G$1" pin="1"/>
+<wire x1="-147.32" y1="-5.08" x2="-144.78" y2="-5.08" width="0.1524" layer="91"/>
+<label x="-144.78" y="-5.08" size="1.778" layer="95"/>
+</segment>
 </net>
 <net name="+5V" class="0">
@@
 <wire x1="238.76" y1="182.88" x2="236.22" y2="182.88" width="0.1524" layer="91"/>
 <label x="236.22" y="182.88" size="1.778" layer="95" rot="R180"/>
-<pinref part="SV1" gate="1" pin="6"/>
+<pinref part="CON3" gate="1" pin="6"/>
 </segment>
 <segment>
@@
 <wire x1="238.76" y1="180.34" x2="236.22" y2="180.34" width="0.1524" layer="91"/>
 <label x="236.22" y="180.34" size="1.778" layer="95" rot="R180"/>
-<pinref part="SV1" gate="1" pin="4"/>
+<pinref part="CON3" gate="1" pin="4"/>
 </segment>
 <segment>
@@
 <wire x1="238.76" y1="177.8" x2="236.22" y2="177.8" width="0.1524" layer="91"/>
 <label x="236.22" y="177.8" size="1.778" layer="95" rot="R180"/>
-<pinref part="SV1" gate="1" pin="2"/>
+<pinref part="CON3" gate="1" pin="2"/>
 </segment>
 <segment>
@@
 </segment>
 </net>
+<net name="SPDIF_DO" class="0">
+<segment>
+<pinref part="CON1" gate="_GPIO-3" pin="24"/>
+<wire x1="-182.88" y1="-22.86" x2="-180.34" y2="-22.86" width="0.1524" layer="91"/>
+<label x="-180.34" y="-22.86" size="1.778" layer="95"/>
+</segment>
+<segment>
+<pinref part="CON4" gate="G$1" pin="2"/>
+<wire x1="-147.32" y1="-2.54" x2="-144.78" y2="-2.54" width="0.1524" layer="91"/>
+<label x="-144.78" y="-2.54" size="1.778" layer="95"/>
+</segment>
+</net>

Commit message: added test points for data lines
fix #7
Parts:
- added BCKAD/DA, DIN1, DOUT1, GND@1, GND@2, LRCKAD/DA, MC, MDI, MDO, MS, SCKI, SPDIF_DO: TPTP10SQ, testpad:TPTP10SQ
Connections:
- net BCKAD/DA: now also BCKAD/DA.TP
- net DIN1: now also DIN1.TP
- net DOUT1: now also DOUT1.TP
- net GND: now also GND@1.TP, GND@2.TP
- net LRCKAD/DA: now also LRCKAD/DA.TP
- net MC: now also MC.TP
- net MDI: now also MDI.TP
- net MDO: now also MDO.TP
- net MS: now also MS.TP
- net SCKI: now also SCKI.TP
- net SPDIF_DO: now also SPDIF_DO.TP
Other:
- moved on the sheet: DIN3, DIN4, DOUT2, DOUT3, OVF, ZERO
